File: Avio-BMS.kicad_pcb (KiCad board)
At the start: 2 copper layers, 80 x 80 mm, 86 parts, among them J1 +3.3V, J10 +7.4V, J2 +3.3V, J3 5077CR-16SMC2-BK-TR, J4 MainBattery, J5 SubBattery, J6 Conn_01x03_Pin, J7 Conn_01x03_Pin, J8 Conn_01x03_Pin, J9 +7.4V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

Commit message: update pcb layoput
Parts:
- moved R3 44.2 mm to (255.1, 153.9), turned to -90 degrees
- moved C17 40.6 mm to (253.7, 156.3)
- moved R2 35.8 mm to (257.8, 153.0), turned to 180 degrees
- moved R1 35.3 mm to (248.4, 155.3), turned to -90 degrees
- moved L1 31.0 mm to (251.1, 144.8)
- moved C4 26.9 mm to (255.1, 150.3), turned to 90 degrees
- moved C1 24.4 mm to (244.6, 150.8), turned to 90 degrees
- moved U1 24.3 mm to (251.2, 152.3), turned to 180 degrees
- moved C5 23.8 mm to (257.1, 150.3), turned to 90 degrees
- moved C2 20.2 mm to (246.6, 150.8), turned to 90 degrees
- moved U3 1.89 mm to (206.9, 86.0)
