File: Avio-BMS.kicad_pcb (KiCad board)
At the start: 2 copper layers, 80 x 80 mm, 90 parts, among them J1 +3.3V, J10 +7.4V, J2 +3.3V, J3 5077CR-16SMC2-BK-TR, J4 MainBattery, J5 SubBattery, J6 Conn_01x03_Pin, J7 Conn_01x03_Pin, J8 Conn_01x03_Pin, J9 +7.4V, Q1 MBT3906DW1, Q2 Si2333DDS-T1-GE3, Q3 Si2333DDS-T1-GE3, Q4 IRF7324, Q5 IRF7324, Q6 IRF7324, Q7 IRF7324, U1 TPS63020DSJR, U2 TPS61088RHLR, U3 LTC4088EDE-TRPBF, U4 LTC4417CGN

Commit message: update pcb
Parts:
- removed the C11 at (215.1, 104.0)
- removed the Q1 at (203.1, 116.2)
- removed the R7 at (122.0, 102.0)
- removed the R8 at (122.0, 99.0)
- removed the R9 at (218.5, 92.5)
- removed the R9 at (215.1, 114.0)
- removed the U3 at (206.9, 86.0)
- added C24: OPT1608, Capacitor_SMD:C_0603_1608Metric_Pad1.08x0.95mm_HandSolder, F.Cu at (121.9, 96.5)
- added C25: 100u, Capacitor_SMD:C_1206_3216Metric_Pad1.33x1.80mm_HandSolder, F.Cu at (124.5, 95.7)
- added C26: OPT3216, Capacitor_SMD:C_1206_3216Metric_Pad1.33x1.80mm_HandSolder, F.Cu at (127.0, 95.7)
- added C27: 0.1u, Capacitor_SMD:C_0603_1608Metric_Pad1.08x0.95mm_HandSolder, F.Cu at (130.2, 96.4)
- added C28: 0.1u, Capacitor_SMD:C_0603_1608Metric_Pad1.08x0.95mm_HandSolder, F.Cu at (81.2, 97.8)
- added C29: 10u, Capacitor_SMD:C_0805_2012Metric_Pad1.18x1.45mm_HandSolder, F.Cu at (141.4, 97.5)
- added C30: 0.1u, Capacitor_SMD:C_0603_1608Metric_Pad1.08x0.95mm_HandSolder, F.Cu at (81.2, 100.3)
- added C31: 10u, Capacitor_SMD:C_0805_2012Metric_Pad1.18x1.45mm_HandSolder, F.Cu at (95.3, 108.2)
- added C32: OPT, Capacitor_SMD:C_0603_1608Metric_Pad1.08x0.95mm_HandSolder, F.Cu at (81.2, 102.8)
- added C33: 10u, Capacitor_SMD:C_0805_2012Metric_Pad1.18x1.45mm_HandSolder, F.Cu at (95.3, 111.2)
- added D3: DF2S232CTC, Diode_SMD:D_0603_1608Metric_Pad1.05x0.95mm_HandSolder, F.Cu at (120.1, 96.5)
- added D4: indi-VBUS, LED_SMD:LED_0603_1608Metric, F.Cu at (114.7, 92.6)
- added D5: indi-charge, LED_SMD:LED_0603_1608Metric, F.Cu at (135.2, 67.3)
- added Q5: Si2333DDS-T1-GE3, Package_TO_SOT_SMD:SOT-23-3, F.Cu at (133.1, 96.4)
- added Q6: Si2333DDS-T1-GE3, Package_TO_SOT_SMD:SOT-23-3, F.Cu at (90.3, 110.7)
- added R17: 5.1k, Resistor_SMD:R_0603_1608Metric_Pad0.98x0.95mm_HandSolder, F.Cu at (121.4, 100.0)
- added R18: 5.1k, Resistor_SMD:R_0603_1608Metric_Pad0.98x0.95mm_HandSolder, F.Cu at (121.4, 101.9)
- added R19: R, Resistor_SMD:R_0603_1608Metric_Pad0.98x0.95mm_HandSolder, F.Cu at (117.3, 90.3)
- added R20: 40k, Resistor_SMD:R_0603_1608Metric_Pad0.98x0.95mm_HandSolder, F.Cu at (131.1, 93.9)
- added R21: 8.2, Resistor_SMD:R_0603_1608Metric_Pad0.98x0.95mm_HandSolder, F.Cu at (81.2, 107.8)
- added R22: 2.94k, Resistor_SMD:R_0603_1608Metric_Pad0.98x0.95mm_HandSolder, F.Cu at (144.1, 87.8)
- added R23: 100k, Resistor_SMD:R_0603_1608Metric_Pad0.98x0.95mm_HandSolder, F.Cu at (135.9, 95.5)
- added R24: 499, Resistor_SMD:R_0603_1608Metric_Pad0.98x0.95mm_HandSolder, F.Cu at (140.9, 89.2)
- added R25: R, Resistor_SMD:R_0603_1608Metric_Pad0.98x0.95mm_HandSolder, F.Cu at (135.9, 70.0)
- added R26: OPT, Resistor_SMD:R_0603_1608Metric_Pad0.98x0.95mm_HandSolder, F.Cu at (85.5, 105.3)
- added R27: 0, Resistor_SMD:R_0603_1608Metric_Pad0.98x0.95mm_HandSolder, F.Cu at (99.8, 79.0)
- added R28: 0, Resistor_SMD:R_0603_1608Metric_Pad0.98x0.95mm_HandSolder, F.Cu at (99.8, 81.5)
- added R29: 0, Resistor_SMD:R_0603_1608Metric_Pad0.98x0.95mm_HandSolder, F.Cu at (99.8, 84.0)
- added TP2: TestPoint, Connector_PinHeader_2.54mm:PinHeader_1x01_P2.54mm_Vertical, F.Cu at (69.8, 113.8)
- added TP3: VBUS, Connector_Pin:Pin_D1.1mm_L8.5mm_W2.5mm_FlatFork, F.Cu at (125.4, 87.9)
- added TP4: BAT-FLOAT4.2V,0.5A, Connector_Pin:Pin_D1.1mm_L8.5mm_W2.5mm_FlatFork, F.Cu at (137.8, 76.4)
- added U4: LTC4088EDE-TRPBF, footprints:DFN-14_DE_LIT, F.Cu at (141.4, 93.4)
- J1: value +3.3V -> MainBattery; footprint Connector_JST:JST_XA_B02B-XASK-1_1x02_P2.50mm_Vertical -> Connector_JST:JST_XA_B03B-XASK-1_1x03_P2.50mm_Vertical
- J2: value +3.3V -> 5077CR-16SMC2-BK-TR; footprint Connector_JST:JST_XA_B02B-XASK-1_1x02_P2.50mm_Vertical -> 5077CR-16SMC2-BK-TR:NELTRON_5077CR-16SMC2-BK-TR
- J3: value 5077CR-16SMC2-BK-TR -> SubBattery; footprint 5077CR-16SMC2-BK-TR:NELTRON_5077CR-16SMC2-BK-TR -> Connector_JST:JST_XA_B03B-XASK-1_1x03_P2.50mm_Vertical
- J4: value MainBattery -> Conn_01x03_Pin; footprint Connector_JST:JST_XA_B02B-XASK-1_1x02_P2.50mm_Vertical -> Connector_PinHeader_2.54mm:PinHeader_1x03_P2.54mm_Vertical
- J5: value SubBattery -> Conn_01x03_Pin; footprint Connector_JST:JST_XA_B02B-XASK-1_1x02_P2.50mm_Vertical -> Connector_PinHeader_2.54mm:PinHeader_1x03_P2.54mm_Vertical
- J7: value Conn_01x03_Pin -> +3.3V; footprint Connector_PinHeader_2.54mm:PinHeader_1x03_P2.54mm_Vertical -> Connector_JST:JST_XA_B02B-XASK-1_1x02_P2.50mm_Vertical
- J8: value Conn_01x03_Pin -> +7.4V; footprint Connector_PinHeader_2.54mm:PinHeader_1x03_P2.54mm_Vertical -> Connector_JST:JST_XA_B02B-XASK-1_1x02_P2.50mm_Vertical
- J9: value +7.4V -> +3.3V
- TP1: value VBUS -> TestPoint; footprint Connector_Pin:Pin_D1.1mm_L8.5mm_W2.5mm_FlatFork -> Connector_PinHeader_2.54mm:PinHeader_1x01_P2.54mm_Vertical
- moved J8 98.5 mm to (144.5, 132.0), turned to 0 degrees
- moved J7 93.9 mm to (153.0, 132.0), turned to 0 degrees
- moved J6 72.8 mm to (153.6, 80.0), turned to 0 degrees
- moved L3 67.2 mm to (148.4, 93.5), turned to 90 degrees
- moved J2 65.0 mm to (117.1, 100.0), turned to -90 degrees
- moved J1 64.3 mm to (147.0, 68.0), turned to 180 degrees
- moved TP1 53.1 mm to (69.8, 109.1)
- moved J3 52.0 mm to (158.0, 68.0), turned to 180 degrees
- moved J10 45.9 mm to (182.0, 105.5), turned to 90 degrees
- moved C13 43.3 mm to (262.5, 76.0)
- moved D2 29.6 mm to (251.9, 134.9)
- moved J5 13.2 mm to (150.0, 80.0), turned to 0 degrees
- moved J4 12.0 mm to (146.4, 80.0), turned to 0 degrees
- moved J9 8.50 mm to (182.0, 97.0)
- renumbered C18 to C1, C6 to C10, C1 to C11, C7 to C12, C2 to C13, C3 to C14, C17 to C15, C15 to C17, C10 to C18, C4 to C19, C19 to C2, C14 to C20, C8 to C21, C5 to C22, C9 to C23, C21 to C3, C22 to C4, C24 to C5, C25 to C6, C27 to C7, C28 to C8, C29 to C9, D3 to D1, D4 to D2, L2 to L1, L1 to L2, Q4 to Q1, Q5 to Q2, Q6 to Q3, Q7 to Q4, R18 to R1, R16 to R10, R1 to R11, R17 to R12, R2 to R13, R3 to R14, R5 to R15, R6 to R16, R19 to R2, R20 to R3, R21 to R4, R22 to R5, R23 to R6, R27 to R7, R28 to R8, R29 to R9, U4 to U1, U1 to U2, U2 to U3
Connections:
- net /DCDC/+3.3V renamed /DCDC3.3V&7.4VOutput/+3.3V
- net /DCDC/7.4V renamed /DCDC3.3V&7.4VOutput/7.4V
- D2 pad 2: Net-(D4-A) -> Net-(D2-A)
- J1 pad 2: /+3.3V -> NTC1
- J10 pad 2: /7.4V -> /出力IO/7.4V
- J4 pad 2: Main-Bat -> D0
- J5 pad 2: V2 -> D1
- J6 pad 2: D0 -> D2
- J7 pad 2: D1 -> /出力IO/+3.3V
- J8 pad 2: D2 -> /出力IO/7.4V
- J9 pad 2: /7.4V -> /出力IO/+3.3V
- R9 pad 1: Net-(D4-A) -> Net-(D2-A)
- TP1 pad 1: VBUS -> GND

Commit message: update pcb ltc4088kitsui
Parts:
- added R12: 0, Resistor_SMD:R_0603_1608Metric_Pad0.98x0.95mm_HandSolder, F.Cu at (148.7, 102.8)
- C2: renamed from C25; value 100u -> 10u; footprint Capacitor_SMD:C_1206_3216Metric_Pad1.33x1.80mm_HandSolder -> Capacitor_SMD:C_0805_2012Metric_Pad1.18x1.45mm_HandSolder
- moved R5 63.8 mm to (141.4, 86.5)
- moved C5 61.5 mm to (141.4, 85.0), turned to 180 degrees
- moved Q2 60.1 mm to (276.7, 77.3)
- moved C10 58.8 mm to (152.9, 99.5), turned to -90 degrees
- moved Q2 58.2 mm to (147.4, 99.5), turned to 180 degrees
- moved C8 56.3 mm to (150.9, 99.5), turned to -90 degrees
- moved R8 35.7 mm to (135.0, 85.0), turned to 90 degrees
- moved R11 33.7 mm to (133.5, 85.0), turned to 90 degrees
- moved R9 32.4 mm to (132.0, 85.0), turned to 90 degrees
- moved R10 22.9 mm to (150.5, 110.0), turned to -90 degrees
- moved L1 17.4 mm to (138.0, 107.5), turned to 0 degrees
- moved TP4 12.3 mm to (150.0, 75.0)
- moved U1 6.13 mm to (140.5, 99.5), turned to 90 degrees
- moved J4 4.64 mm to (150.3, 82.5)
- moved J5 4.64 mm to (153.9, 82.5)
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- renumbered C24 to C1, C33 to C10, C1 to C11, C2 to C12, C3 to C13, C4 to C14, C5 to C15, C6 to C16, C7 to C17, C8 to C18, C9 to C19, C10 to C20, C11 to C21, C12 to C22, C13 to C23, C14 to C24, C15 to C25, C16 to C26, C17 to C27, C18 to C28, C19 to C29, C26 to C3, C20 to C30, C21 to C31, C22 to C32, C23 to C33, C27 to C4, C28 to C5, C29 to C6, C30 to C7, C31 to C8, C32 to C9, D3 to D1, D4 to D2, D5 to D3, D1 to D4, D2 to D5, L3 to L1, L1 to L2, L2 to L3, Q5 to Q1, Q6 to Q2, Q1 to Q3, Q2 to Q4, Q3 to Q5, Q4 to Q6, R17 to R1, R24 to R10, R29 to R11, R25 to R13, R26 to R14, R1 to R15, R2 to R16, R3 to R17, R4 to R18, R5 to R19, R18 to R2, R6 to R20, R7 to R21, R8 to R22, R9 to R23, R10 to R24, R11 to R25, R12 to R26, R13 to R27, R14 to R28, R15 to R29, R19 to R3, R16 to R30, R20 to R4, R21 to R5, R22 to R6, R23 to R7, R27 to R8, R28 to R9, U4 to U1, U1 to U2, U2 to U3, U3 to U4
Connections:
- C10 pad 1: Main-Bat -> V1
- C8 pad 1: Main-Bat -> V1
- D2 pad 2: Net-(D4-A) (its old number) -> Net-(D2-A)
- D3 pad 2: Main-Bat -> V1
- D5 pad 2: Net-(D2-A) -> Net-(D5-A)
- L1 pad 2: Main-Bat -> V1
- Q2 pad 1: /Li-ionBatteryCharger,PowerPath/GATE -> Net-(Q2-G)
- Q2 pad 2: Main-Bat -> V1
- R23 pad 1: Net-(D2-A) -> Net-(D5-A)
- R3 pad 1: Net-(D4-A) (its old number) -> Net-(D2-A)
- U1 pad 10: Main-Bat -> V1
- U1 pad 3: Main-Bat -> V1
Routing:
- net NTC2: track 0.00 -> 43.4 mm
- net VBUS: track 0.00 -> 37.1 mm
- net D2: track 0.00 -> 34.4 mm, vias 0 -> 1
- net V_{IN}: track 0.00 -> 30.3 mm
- net NTC1: track 0.00 -> 30.1 mm
- net NTC: track 0.00 -> 25.4 mm, vias 0 -> 2
- net V1: track 0.00 -> 23.8 mm
- net D1: track 0.00 -> 23.5 mm, vias 0 -> 1
- net D0: track 0.00 -> 21.3 mm, vias 0 -> 1
- net Net-(U1-SW): track 0.00 -> 14.1 mm
- net /Li-ionBatteryCharger,PowerPath/GATE: track 0.00 -> 12.6 mm, vias 0 -> 2
- net Net-(J2-CC1): track 0.00 -> 2.82 mm
- net Net-(Q2-G): track 0.00 -> 2.37 mm
- net Net-(J2-CC2): track 0.00 -> 2.36 mm
- net Net-(D2-A): track 0.00 -> 2.31 mm
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- added copper zone on F.Cu, net V1

Commit message: update pcb
Parts:
- removed the C12 at (213.0, 87.0)
- removed the C20 at (222.0, 84.0)
- removed the C23 at (218.0, 87.0)
- removed the Q3 at (232.5, 85.5)
- removed the R10 at (214.0, 120.0)
- removed the R11 at (204.1, 79.0)
- removed the R12 at (201.5, 71.5)
- removed the R13 at (202.5, 84.5)
- removed the R14 at (85.5, 105.3)
- removed the R14 at (204.0, 89.0)
- removed the TP2 at (231.7, 92.7)
- added R14: OPT, Resistor_SMD:R_0603_1608Metric_Pad0.98x0.95mm_HandSolder, F.Cu at (135.6, 77.7)
- moved TP2 93.9 mm to (161.2, 135.1)
- moved C9 63.8 mm to (139.3, 76.5)
- moved C7 62.2 mm to (139.3, 78.0)
- moved TP1 57.6 mm to (122.3, 85.4)
- moved J5 32.4 mm to (132.8, 107.1), turned to 180 degrees
- moved J4 32.4 mm to (129.2, 107.1), turned to 180 degrees
- moved J6 32.4 mm to (136.4, 107.1), turned to 180 degrees
- moved R10 21.2 mm to (145.8, 89.3), turned to 45 degrees
- moved C10 17.8 mm to (146.6, 82.8), turned to -45 degrees
- moved C8 16.3 mm to (145.2, 84.2), turned to -45 degrees
- moved C5 15.4 mm to (131.0, 96.4)
- moved R12 15.1 mm to (144.7, 88.3), turned to 45 degrees
- moved TP4 14.7 mm to (135.8, 71.3)
- moved Q2 13.6 mm to (142.7, 86.7), turned to -135 degrees
- moved R5 12.1 mm to (134.4, 96.4), turned to 180 degrees
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Routing:
- net Main-Bat: track 2.24 -> 29.0 mm, vias 1 -> 0
- net D1: track 23.5 -> 1.50 mm
- net V_{IN}: track 30.3 -> 9.99 mm
- net D0: track 21.3 -> 2.70 mm
- net D2: track 34.4 -> 16.3 mm
- net NTC: track 25.4 -> 17.2 mm
- net Net-(U1-CLPROG): track 0.00 -> 8.17 mm, vias 0 -> 2
- net Net-(U1-C/X): track 0.00 -> 7.02 mm
- net /Li-ionBatteryCharger,PowerPath/GATE: track 12.6 -> 6.18 mm, vias 2 -> 0
- net Net-(Q1-G): track 0.00 -> 5.92 mm
- net VBUS: track 37.1 -> 40.3 mm
- net V1: track 23.8 -> 26.9 mm, vias 0 -> 33
- net Net-(Q2-G): track 2.37 -> 0.00 mm
- net NTC1: track 30.1 -> 28.4 mm
- net Net-(C5-Pad1): track 0.00 -> 1.56 mm
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- added copper zone on B.Cu, net V1

Commit message: ltc4417
Parts:
- removed Q5, Q6: IRF7324, Package_SO:SOIC-8_3.9x4.9mm_P1.27mm
- moved Q4 116.6 mm to (152.4, 77.8), turned to 90 degrees
- moved D5 115.7 mm to (137.9, 70.7), turned to 45 degrees
- moved R23 113.8 mm to (139.2, 71.9), turned to -135 degrees
- moved D4 113.8 mm to (135.3, 73.3), turned to 45 degrees
- moved R22 112.0 mm to (136.4, 74.4), turned to -135 degrees
- moved Q3 107.1 mm to (145.6, 77.8), turned to 90 degrees
- moved R18 105.0 mm to (138.7, 89.2)
- moved C11 101.5 mm to (150.5, 85.8), turned to 0 degrees
- moved R15 99.7 mm to (141.1, 86.9)
- moved R16 99.7 mm to (141.1, 90.2)
- moved R17 99.7 mm to (141.1, 93.5)
- moved R19 99.4 mm to (138.7, 92.5)
- moved C12 99.4 mm to (153.0, 89.4), turned to 0 degrees
- moved R21 97.5 mm to (146.0, 101.8), turned to 0 degrees
- moved JP1 96.7 mm to (146.6, 99.5)
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Connections:
- C16 pad 2: Net-(Q5A-S1) -> Net-(Q3B-S2)
- Q3 pad 3: (no net) -> Net-(Q3B-S2)
- Q3 pad 4: (no net) -> Net-(Q3B-G2)
- Q3 pad 5: (no net) -> VCC
- Q3 pad 6: (no net) -> VCC
- Q4 pad 1: Net-(Q3A-S1) -> Net-(Q3B-S2)
- Q4 pad 2: Net-(Q3A-G1) -> Net-(Q3B-G2)
- Q4 pad 3: (no net) -> Net-(Q3A-S1)
- Q4 pad 4: (no net) -> Net-(Q3A-G1)
- Q4 pad 5: (no net) -> VCC
- Q4 pad 6: (no net) -> VCC
- Q4 pad 7: VCC -> V2
- Q4 pad 8: VCC -> V2
- U2 pad 18: Net-(Q5A-G1) -> Net-(Q3B-G2)
- U2 pad 19: Net-(Q5A-S1) -> Net-(Q3B-S2)
Routing:
- net V2: track 0.00 -> 56.6 mm, vias 0 -> 1
- net V1: track 26.9 -> 72.4 mm, vias 33 -> 27
- net /Li-ionBatteryCharger,PowerPath/*CHRG: track 0.00 -> 41.4 mm, vias 0 -> 4
- net V_{IN}: track 9.99 -> 32.8 mm, vias 0 -> 1
- net D0: track 2.70 -> 20.3 mm, vias 1 -> 2
- net D1: track 1.50 -> 17.9 mm, vias 1 -> 2
- net Net-(Q3A-G1): track 0.00 -> 5.31 mm, vias 0 -> 1
- net OV2: track 0.00 -> 5.00 mm
- net UV2: track 0.00 -> 4.69 mm, vias 0 -> 1
- net OV1: track 0.00 -> 4.65 mm
- net Main-Bat: track 29.0 -> 25.3 mm
- net Net-(Q3B-S2): track 0.00 -> 3.17 mm
- net Net-(Q3A-S1): track 0.00 -> 3.07 mm
- net NTC: track 17.2 -> 20.2 mm
- net ~{VALID2}: track 0.00 -> 2.90 mm, vias 0 -> 2
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
Commit message: update
Parts:
- moved C25 122.7 mm to (154.2, 84.6)
- moved C29 122.7 mm to (155.5, 78.6)
- moved C32 122.7 mm to (157.5, 78.6)
- moved L3 122.7 mm to (151.5, 73.1)
- moved R25 122.7 mm to (148.8, 83.6)
- moved R27 122.7 mm to (158.2, 81.3)
- moved R28 122.7 mm to (155.5, 82.2)
- moved U3 122.7 mm to (151.6, 80.6)
- moved C21 122.6 mm to (145.0, 79.3)
- moved C23 122.6 mm to (147.0, 79.3)
- moved REF** 56.5 mm to (187.5, 101.5), turned to 180 degrees
- moved D2 55.2 mm to (171.3, 131.7), turned to -135 degrees
- moved REF** 52.5 mm to (151.5, 137.5), turned to 180 degrees
- moved R3 52.2 mm to (167.8, 131.5), turned to 135 degrees
- moved J2 51.4 mm to (174.8, 124.7), turned to 45 degrees
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Routing:
- net VCC: track 0.00 -> 62.8 mm
- net ~{VALID1}: track 1.68 -> 37.8 mm, vias 1 -> 2
- net Net-(Q3B-S2): track 3.17 -> 35.1 mm, vias 0 -> 2
- net Net-(Q3A-S1): track 3.07 -> 32.9 mm, vias 0 -> 2
- net Net-(Q3A-G1): track 5.31 -> 34.5 mm, vias 1 -> 2
- net ~{VALID2}: track 2.90 -> 29.3 mm
- net Net-(Q3B-G2): track 0.00 -> 23.6 mm, vias 0 -> 2
- net V1: track 72.4 -> 94.8 mm
- net Net-(JP1-C): track 0.00 -> 10.3 mm
- net Net-(U3-L1_8): track 0.00 -> 7.33 mm
- net Net-(U3-L2_6): track 0.00 -> 7.17 mm
- net V2: track 56.6 -> 63.6 mm, vias 1 -> 3
- net UV1: track 1.48 -> 5.89 mm
- net UV2: track 4.69 -> 8.06 mm, vias 1 -> 2
- net Net-(JP1-A): track 0.00 -> 2.35 mm
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
Commit message: update pcb
Parts:
- removed the C13 at (262.5, 76.0)
- removed C3: OPT3216, Capacitor_SMD:C_1206_3216Metric_Pad1.33x1.80mm_HandSolder
- removed the D1 at (229.2, 113.2)
- removed the D2 at (251.9, 134.9)
- removed the Q2 at (276.7, 77.3)
- removed the R15 at (219.4, 114.0)
- removed R28: 137k, Resistor_SMD:R_0603_1608Metric_Pad0.98x0.95mm_HandSolder
- removed the R4 at (210.5, 108.9)
- removed U3: TPS63020DSJR, TPS63020DSJR:IC_TPS63020DSJR
- added C34: 22u, Capacitor_SMD:C_0805_2012Metric_Pad1.18x1.45mm_HandSolder, F.Cu at (133.6, 72.4)
- added C35: 22u, Capacitor_SMD:C_0805_2012Metric_Pad1.18x1.45mm_HandSolder, F.Cu at (135.0, 70.9)
- added C36: 0.1u, Capacitor_SMD:C_0603_1608Metric_Pad1.08x0.95mm_HandSolder, F.Cu at (126.6, 80.6)
- added D6: LED, LED_SMD:LED_0603_1608Metric, F.Cu at (128.3, 84.6)
- added U5: TPS63021DSJR, TPS63021DSJR:IC_TPS63021DSJR, F.Cu at (129.4, 79.4)
- C1: value OPT1608 -> 10u; footprint Capacitor_SMD:C_0603_1608Metric_Pad1.08x0.95mm_HandSolder -> Capacitor_SMD:C_0805_2012Metric_Pad1.18x1.45mm_HandSolder
- C21, C23, C29, C32: value 10u -> 22u
- L3: value 1.5u -> 1u; footprint Inductor_SMD:L_Vishay_IHLP-1616 -> Inductor_SMD:L_1210_3225Metric_Pad1.42x2.65mm_HandSolder
- R27: value 768k -> 10M
- moved L2 123.0 mm to (142.7, 69.9)
- moved C20 88.9 mm to (143.7, 78.2)
- moved C22 88.9 mm to (141.7, 78.2)
- moved C24 88.9 mm to (147.2, 78.2)
- moved C27 88.9 mm to (154.5, 76.7)
- moved C28 88.9 mm to (162.5, 76.7)
- moved C30 88.9 mm to (160.5, 76.7)
- moved C31 88.9 mm to (156.5, 76.7)
- moved C33 88.9 mm to (158.5, 76.7)
- moved R24 88.9 mm to (147.2, 73.3)
- moved R26 88.9 mm to (153.7, 71.8)
- moved U4 88.9 mm to (150.5, 75.2)
- moved C26 88.9 mm to (148.7, 79.7)
- moved R29 88.9 mm to (158.9, 73.7)
- moved R30 88.9 mm to (156.5, 72.7)
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Connections:
- net /DCDC3.3V&7.4VOutput/7.4V renamed +6V
- C1 pad 1: VBUS -> Net-(C1-Pad1)
- C15 pad 1: GND -> Net-(Q3A-S1)
- C15 pad 2: Net-(Q3A-S1) -> GND
- C29 pad 1: /DCDC3.3V&7.4VOutput/+3.3V -> +3.3V
- C32 pad 1: /DCDC3.3V&7.4VOutput/+3.3V -> +3.3V
- J2 pad S1: Net-(J2-SHIELD-PadS1) -> Net-(C1-Pad1)
- J2 pad S2: Net-(J2-SHIELD-PadS1) -> Net-(C1-Pad1)
- J2 pad S3: Net-(J2-SHIELD-PadS1) -> Net-(C1-Pad1)
- J2 pad S4: Net-(J2-SHIELD-PadS1) -> Net-(C1-Pad1)
- J7 pad 2: /出力IO/+3.3V -> +3.3V
- J9 pad 2: /出力IO/+3.3V -> +3.3V
- R25 pad 2: /DCDC3.3V&7.4VOutput/+3.3V -> +3.3V
- R27 pad 1: /DCDC3.3V&7.4VOutput/+3.3V -> GND
- R27 pad 2: Net-(U3-FB) -> Net-(C1-Pad1)
Routing:
- net +3.3V: track 0.00 -> 71.3 mm
- net /出力IO/7.4V: track 0.00 -> 57.1 mm
- net VCC: track 62.8 -> 91.5 mm
- net Net-(C1-Pad1): track 0.00 -> 20.8 mm
- net +6V: track 0.00 -> 11.6 mm
- net Net-(D6-K): track 0.00 -> 4.32 mm
- net Net-(U5-L1_8): track 7.33 -> 4.80 mm
- net Net-(U5-L2_6): track 7.17 -> 4.76 mm
- net Net-(U5-EN): track 0.00 -> 2.13 mm
- net Net-(D6-A): track 0.00 -> 1.69 mm

Commit message: update pcb sch
Parts:
- removed J4: Conn_01x03_Pin, Connector_PinHeader_2.54mm:PinHeader_1x03_P2.54mm_Vertical
- added C3: 100u, Capacitor_SMD:C_1206_3216Metric_Pad1.33x1.80mm_HandSolder, F.Cu at (205.8, 109.1)
- C6: value 10u -> 100u; footprint Capacitor_SMD:C_0805_2012Metric_Pad1.18x1.45mm_HandSolder -> Capacitor_SMD:C_1206_3216Metric_Pad1.33x1.80mm_HandSolder
- J10, J8: value +7.4V -> +6V
- moved C6 0.51 mm to (155.5, 107.9)
Connections:
- net V_{IN} renamed /Li-ionBatteryCharger,PowerPath/V_{IN}
- J10 pad 2: /出力IO/7.4V -> +6V
- J5 pad 2: D1 -> /Li-ionBatteryCharger,PowerPath/D1
- J6 pad 2: D2 -> /Li-ionBatteryCharger,PowerPath/D1
- J8 pad 2: /出力IO/7.4V -> +6V
- U1 pad 13: D0 -> GND
- U1 pad 14: D1 -> /Li-ionBatteryCharger,PowerPath/D1
- U1 pad 4: D2 -> /Li-ionBatteryCharger,PowerPath/D2
Routing:
- net +6V: track 11.6 -> 100.1 mm
- net /出力IO/7.4V: track 57.1 -> 0.00 mm
- net D0: track 20.3 -> 0.00 mm, vias 2 -> 0
- net D1: track 17.9 -> 0.00 mm, vias 2 -> 0
- net /Li-ionBatteryCharger,PowerPath/D1: track 0.00 -> 17.9 mm, vias 0 -> 2
- net D2: track 16.3 -> 0.00 mm, vias 1 -> 0
- net (no net): track 0.00 -> 16.3 mm, vias 0 -> 1
- net FB_{TPS61088}: track 0.00 -> 6.20 mm
- net Net-(U4-FSW): track 0.00 -> 2.41 mm
- net /Li-ionBatteryCharger,PowerPath/V_{IN}: track 32.8 -> 30.7 mm
- net Net-(U4-SS): track 0.00 -> 1.94 mm
- net Net-(U4-ILIM): track 0.00 -> 1.88 mm
- net ~{VALID1}: track 37.8 -> 36.3 mm
- net ~{VALID2}: track 29.3 -> 30.7 mm

Commit message: ad datasheet
Parts:
- added TP5: 6V, Connector_Pin:Pin_D1.1mm_L8.5mm_W2.5mm_FlatFork, F.Cu at (138.4, 59.7)
- added TP6: 3.3V, Connector_Pin:Pin_D1.1mm_L8.5mm_W2.5mm_FlatFork, F.Cu at (129.7, 74.8)
- moved C6 37.2 mm to (168.9, 104.5), turned to -45 degrees
- moved R8 18.0 mm to (175.9, 107.1), turned to 135 degrees
- moved R9 14.0 mm to (173.8, 109.2)
- moved R10 14.0 mm to (174.9, 108.1)
- moved R12 14.0 mm to (172.8, 110.2)
- moved TP1 13.6 mm to (181.2, 107.3)
- moved C4 11.9 mm to (167.2, 106.1)
- moved C20 11.7 mm to (155.3, 76.1)
- moved C25 11.7 mm to (138.1, 78.6)
- moved C3 11.7 mm to (173.0, 99.3)
- moved D1 11.7 mm to (182.9, 93.2)
- moved R14 11.7 mm to (167.9, 118.3)
- moved R19 11.7 mm to (147.8, 106.3)
- moved R26 11.7 mm to (165.3, 69.7)
- moved R5 11.7 mm to (169.6, 99.3)
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- renumbered C36 to C25, C25 to C26, C26 to C27, C27 to C28, C28 to C29, C4 to C3, C29 to C30, C30 to C31, C31 to C33, C33 to C35, C35 to C36, C6 to C4, C3 to C6, J5 to J4, J6 to J5, J7 to J6, J8 to J7, J9 to J8, J10 to J9, R27 to R1, R9 to R10, R10 to R11, R11 to R12, R12 to R13, R13 to R14, R14 to R15, R15 to R16, R16 to R17, R17 to R18, R18 to R19, R1 to R2, R19 to R20, R20 to R21, R21 to R22, R22 to R23, R23 to R24, R24 to R25, R29 to R27, R30 to R28, R25 to R29, R2 to R3, R3 to R4, R4 to R5, R5 to R6, R6 to R7, R7 to R8, R8 to R9, U5 to U3
Connections:
- net Net-(U4-SW_4) renamed /DCDC3.3V&7.4VOutput/SW_4567
Routing:
- net /Li-ionBatteryCharger,PowerPath/V_{IN}: track 30.7 -> 37.2 mm
- net NTC: track 20.2 -> 22.2 mm
- net /DCDC3.3V&7.4VOutput/SW_4567: track 0.00 -> 0.88 mm
- net Net-(U1-SW): track 14.9 -> 14.4 mm
- added copper zone on F.Cu, net /DCDC3.3V&7.4VOutput/SW_4567
