File: DCDC.kicad_sch (KiCad schematic)
At the start: 25 parts, among them U1 TPS63020DSJR, U2 TPS61088RHLR

Commit message: update pcb
Parts:
- renumbered C6 to C10, C1 to C11, C7 to C12, C2 to C13, C3 to C14, C17 to C15, C15 to C17, C10 to C18, C4 to C19, C14 to C20, C8 to C21, C5 to C22, C9 to C23, L2 to L1, L1 to L2, R16 to R10, R1 to R11, R17 to R12, R2 to R13, R3 to R14, R5 to R15, R6 to R16, U1 to U2, U2 to U3

Commit message: update pcb ltc4088kitsui
Parts:
- renumbered C10 to C20, C11 to C21, C12 to C22, C13 to C23, C14 to C24, C15 to C25, C16 to C26, C17 to C27, C18 to C28, C19 to C29, C20 to C30, C21 to C31, C22 to C32, C23 to C33, L1 to L2, L2 to L3, R10 to R24, R11 to R25, R12 to R26, R13 to R27, R14 to R28, R15 to R29, R16 to R30, U2 to U3, U3 to U4

Commit message: update pcb
Parts:
- removed R27: 768k, Resistor_SMD:R_0603_1608Metric_Pad0.98x0.95mm_HandSolder, symbol Device:R_Small
- removed R28: 137k, Resistor_SMD:R_0603_1608Metric_Pad0.98x0.95mm_HandSolder, symbol Device:R_Small
- removed U3: TPS63020DSJR, TPS63020DSJR:IC_TPS63020DSJR, symbol TPS63020DSJR:TPS63020DSJR
- added C34, C35: 22u, Capacitor_SMD:C_0805_2012Metric_Pad1.18x1.45mm_HandSolder, symbol Device:C
- added C36: 0.1u, Capacitor_SMD:C_0603_1608Metric_Pad1.08x0.95mm_HandSolder, symbol Device:C_Small
- added D6: LED, LED_SMD:LED_0603_1608Metric, symbol Device:LED
- added U5: TPS63021DSJR, TPS63021DSJR:IC_TPS63021DSJR, symbol TPS63021DSJR:TPS63021DSJR
- C21, C23, C29, C32: value 10u -> 22u
- L3: value 1.5u -> 1u; footprint Inductor_SMD:L_Vishay_IHLP-1616 -> Inductor_SMD:L_1210_3225Metric_Pad1.42x2.65mm_HandSolder
Connections:
- net +3.3V: now also C34.1, C35.1, U5.3 (FB), U5.4 (VOUT_4), U5.5 (VOUT_5)
- net GND: now also C34.2, C35.2, C36.2, U5.13 (PS/SYNC), U5.15 (PGND), U5.2 (GND)
- net VCC: now also C36.1, U5.10 (VIN_10), U5.11 (VIN_11)
- net at C25.1: now also U5.1 (VINA), U5.12 (EN)
- net at R25.1: now also D6.2 (A)
- net at L3.1: now also U5.8 (L1_8), U5.9 (L1_9)
- net at L3.2: now also U5.6 (L2_6), U5.7 (L2_7)
- net 7.4V renamed +6V
- new net: D6.1 (K), U5.14 (PG)
Other:
- note added: "3.3V MCU/Sensor"
- moved on the sheet: C20, C21, C22, C23, C24, C25, C26, C27, C28, C29, C30, C31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

Commit message: ad datasheet
Parts:
- added C37: 0.1u, Capacitor_SMD:C_0603_1608Metric_Pad1.08x0.95mm_HandSolder, symbol Device:C_Small
- added TP5: 6V, Connector_Pin:Pin_D1.1mm_L8.5mm_W2.5mm_FlatFork, symbol Connector:TestPoint
- added TP6: 3.3V, Connector_Pin:Pin_D1.1mm_L8.5mm_W2.5mm_FlatFork, symbol Connector:TestPoint
- renumbered C36 to C25, C25 to C26, C26 to C27, C27 to C28, C28 to C29, C29 to C30, C30 to C31, C31 to C33, C33 to C35, C35 to C36, R24 to R25, R29 to R27, R30 to R28, R25 to R29, U5 to U3
Connections:
- net +3.3V: now also TP6.1
- net +6V: now also TP5.1
- net SW_4567: now reaches L2.2, R25.1, U4.4 (SW_7), U4.5 (SW_4), U4.6 (SW_5), U4.7 (SW_6)
- net SW_4567: now also C37.2
- net at U4.8 (BOOT): now also C37.1

Commit message: update pcb
Parts:
- added C38: 1u, Capacitor_SMD:C_0603_1608Metric_Pad1.08x0.95mm_HandSolder, symbol Device:C_Small
- added C39: 43p, Capacitor_SMD:C_0603_1608Metric_Pad1.08x0.95mm_HandSolder, symbol Device:C_Small
- added C40: 1n, Capacitor_SMD:C_0603_1608Metric_Pad1.08x0.95mm_HandSolder, symbol Device:C_Small
- added R30: 28.7k, Resistor_SMD:R_0603_1608Metric_Pad0.98x0.95mm_HandSolder, symbol Device:R_Small
- C27: value C -> 8.2n
- R26: value R -> 115k
Connections:
- net EN_{TPS61088}: now also U4.1 (VCC_{TPS61088}), C38.1
- net GND: now also U4.13 (MODE), C38.2, C39.1, C40.1
- net COMP_{TPS61088}: now reaches U4.18 (COMP)
- net COMP_{TPS61088}: now also C39.2, R30.1
- new net: C40.2, R30.2
Other:
- note added: "PWMmodeで使用する"
- moved on the sheet: C28, C29, C31, C33, C35, R26, R27, R28, TP5

Commit message: update
Changed lines of the file:
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@@
+		)
+	)
+	(text_box "11V->R27=976k, R28=120k\n6V->R27=470k, R28=118k\n"
+		(exclude_from_sim no)
+		(at 194.31 134.62 0)
+		(size 30.48 5.08)
+		(stroke
+			(width 0)
+			(type default)
+		)
+		(fill
+			(type none)
+		)
+		(effects
+			(font
+				(size 1.27 1.27)
+			)
+			(justify left top)
 		)
 	)
