File: DCDC.kicad_sch (KiCad schematic)
At the start: 34 parts, among them U3 TPS63021DSJR, U4 TPS61088RHLR

Commit message: 値の更新とテキストボックスの修正; LTC4088およびLTC4417の新しいテキスト追加
Parts:
- R27: value R -> 221k
- R28: value R -> 56k
Changed lines of the file:
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@@
 		)
 	)
-	(text_box "11V->R27=976k, R28=120k\n6V->R27=470k, R28=118k\n"
+	(text_box "R27=(V_{OUT}-V{REF}*R28)/V{REF}\nV{REF}=1.204V(Modeによって少し変わる)\nR28は56kOhmが標準的に使われる\n(Example)\n11V->R27=976k, R28=120k\n6V->R27=223k, R28=56k\n"
 		(exclude_from_sim no)
-		(at 194.31 134.62 0)
-		(size 30.48 5.08)
+		(at 198.12 134.62 0)
+		(size 43.18 13.97)
 		(stroke
 			(width 0)
@@
 			)
 		)
-		(property "Value" "R"
+		(property "Value" "56k"
 			(at 185.42 139.6999 0)
 			(effects
@@
 			)
 		)
-		(property "Value" "R"
+		(property "Value" "221k"
 			(at 185.42 126.9999 0)
 			(effects
