File: Output.kicad_sch (KiCad schematic)
At the start: 4 parts, among them J1 +3.3V, J10 +7.4V, J2 +7.4V, J9 +3.3V

Commit message: update pcb
Parts:
- renumbered J1 to J7, J2 to J8
Changed lines of the file:
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@@
 		(dnp no)
 		(fields_autoplaced yes)
-		(property "Reference" "#PWR013"
+		(property "Reference" "#PWR055"
 			(at 128.27 90.17 0)
 			(effects
@@
 			(project "Avio-BMS"
 				(path "/14e0994b-afc2-4c10-b50d-3efcc006980d/b371f4c8-5a59-4bdf-859b-16f2afd474be"
-					(reference "#PWR013")
+					(reference "#PWR055")
 					(unit 1)
 				)
@@
 		(dnp no)
 		(fields_autoplaced yes)
-		(property "Reference" "#PWR046"
+		(property "Reference" "#PWR056"
 			(at 128.27 111.76 0)
 			(effects
@@
 			(project "Avio-BMS"
 				(path "/14e0994b-afc2-4c10-b50d-3efcc006980d/b371f4c8-5a59-4bdf-859b-16f2afd474be"
-					(reference "#PWR046")
+					(reference "#PWR056")
 					(unit 1)
 				)
@@
 		(on_board yes)
 		(dnp no)
-		(property "Reference" "J1"
+		(property "Reference" "J7"
 			(at 142.24 90.1701 0)
 			(effects
@@
 			(project "Avio-BMS"
 				(path "/14e0994b-afc2-4c10-b50d-3efcc006980d/b371f4c8-5a59-4bdf-859b-16f2afd474be"
-					(reference "J1")
+					(reference "J7")
 					(unit 1)
 				)
@@
 		(dnp no)
 		(fields_autoplaced yes)
-		(property "Reference" "#PWR053"
+		(property "Reference" "#PWR058"
 			(at 149.86 111.76 0)
 			(effects
@@
 			(project "Avio-BMS"
 				(path "/14e0994b-afc2-4c10-b50d-3efcc006980d/b371f4c8-5a59-4bdf-859b-16f2afd474be"
-					(reference "#PWR053")
+					(reference "#PWR058")
 					(unit 1)
 				)
@@
 		(on_board yes)
 		(dnp no)
-		(property "Reference" "J2"
+		(property "Reference" "J8"
 			(at 142.24 111.7601 0)
 			(effects
@@
 			(project "Avio-BMS"
 				(path "/14e0994b-afc2-4c10-b50d-3efcc006980d/b371f4c8-5a59-4bdf-859b-16f2afd474be"
-					(reference "J2")
+					(reference "J8")
 					(unit 1)
 				)
@@
 		(dnp no)
 		(fields_autoplaced yes)
-		(property "Reference" "#PWR050"
+		(property "Reference" "#PWR057"
 			(at 149.86 90.17 0)
 			(effects
@@
 			(project "Avio-BMS"
 				(path "/14e0994b-afc2-4c10-b50d-3efcc006980d/b371f4c8-5a59-4bdf-859b-16f2afd474be"
-					(reference "#PWR050")
-					(unit 1)
-				)
+					(reference "#PWR057")
+					(unit 1)
+				)

Commit message: update pcb
Other:
- moved on the sheet: J9
Changed lines of the file:
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@@
 		)
 	)
-	(label "+3.3V"
-		(at 156.21 87.63 180)
+	(label "7.4V"
+		(at 156.21 109.22 180)
 		(fields_autoplaced yes)
 		(effects
@@
 		)
 	)
-	(label "+3.3V"
-		(at 134.62 87.63 180)
-		(fields_autoplaced yes)
-		(effects
-			(font
-				(size 1.27 1.27)
-			)
-			(justify right bottom)
-		)
-	)
-	(label "7.4V"
-		(at 156.21 109.22 180)
-		(fields_autoplaced yes)
-		(effects
-			(font
-				(size 1.27 1.27)
-			)
-			(justify right bottom)
-		)
-	)
 	(symbol
 		(lib_id "power:GND")
@@
 				(path "/14e0994b-afc2-4c10-b50d-3efcc006980d/b371f4c8-5a59-4bdf-859b-16f2afd474be"
 					(reference "#PWR056")
+					(unit 1)
+				)
+			)
+		)
+	)
+	(symbol
+		(lib_id "power:+3.3V")
+		(at 134.62 87.63 90)
+		(unit 1)
+		(exclude_from_sim no)
+		(in_bom yes)
+		(on_board yes)
+		(dnp no)
+		(fields_autoplaced yes)
+		(property "Reference" "#PWR061"
+			(at 138.43 87.63 0)
+			(effects
+				(font
+					(size 1.27 1.27)
+				)
+				(hide yes)
+			)
+		)
+		(property "Value" "+3.3V"
+			(at 130.81 87.6299 90)
+			(effects
+				(font
+					(size 1.27 1.27)
+				)
+				(justify left)
+			)
+		)
+		(property "Footprint" ""
+			(at 134.62 87.63 0)
+			(effects
+				(font
+					(size 1.27 1.27)
+				)
+				(hide yes)
+			)
+		)
+		(property "Datasheet" ""
+			(at 134.62 87.63 0)
+			(effects
+				(font
+					(size 1.27 1.27)
+				)
+				(hide yes)
+			)
+		)
+		(property "Description" "Power symbol creates a global label with name \"+3.3V\""
+			(at 134.62 87.63 0)
+			(effects
+				(font
+					(size 1.27 1.27)
+				)
+				(hide yes)
+			)
+		)
+		(pin "1"
+		)
+		(instances
+			(project "Avio-BMS"
+				(path "/14e0994b-afc2-4c10-b50d-3efcc006980d/b371f4c8-5a59-4bdf-859b-16f2afd474be"
+					(reference "#PWR061")
+					(unit 1)
+				)
+			)
+		)
+	)
+	(symbol
+		(lib_id "power:+3.3V")
+		(at 163.83 87.63 90)
+		(unit 1)
+		(exclude_from_sim no)
+		(in_bom yes)
+		(on_board yes)
+		(dnp no)
+		(fields_autoplaced yes)
+		(property "Reference" "#PWR062"
+			(at 167.64 87.63 0)
+			(effects
+				(font
+					(size 1.27 1.27)
+				)
+				(hide yes)
+			)
+		)
+		(property "Value" "+3.3V"
+			(at 160.02 87.6299 90)
+			(effects
+				(font
+					(size 1.27 1.27)
+				)
+				(justify left)
+			)
+		)
+		(property "Footprint" ""
+			(at 163.83 87.63 0)
+			(effects
+				(font
+					(size 1.27 1.27)
+				)
+				(hide yes)
+			)
+		)
+		(property "Datasheet" ""
+			(at 163.83 87.63 0)
+			(effects
+				(font
+					(size 1.27 1.27)
+				)
+				(hide yes)
+			)
+		)
+		(property "Description" "Power symbol creates a global label with name \"+3.3V\""
+			(at 163.83 87.63 0)
+			(effects
+				(font
+					(size 1.27 1.27)
+				)
+				(hide yes)
+			)
+		)
+		(pin "1"
+		)
+		(instances
+			(project "Avio-BMS"
+				(path "/14e0994b-afc2-4c10-b50d-3efcc006980d/b371f4c8-5a59-4bdf-859b-16f2afd474be"
+					(reference "#PWR062")
 					(unit 1)
 				)
@@
 	(symbol
 		(lib_id "power:GND")
-		(at 156.21 90.17 270)
+		(at 163.83 90.17 270)
 		(unit 1)
 		(exclude_from_sim no)
@@
 		(fields_autoplaced yes)
 		(property "Reference" "#PWR057"
-			(at 149.86 90.17 0)
+			(at 157.48 90.17 0)
 			(effects
 				(font
@@
 		)
 		(property "Value" "GND"
-			(at 152.4 90.1699 90)
+			(at 160.02 90.1699 90)
 			(effects
 				(font
@@
 		)
 		(property "Footprint" ""
-			(at 156.21 90.17 0)
+			(at 163.83 90.17 0)
 			(effects
 				(font
@@
 		)
 		(property "Datasheet" ""
-			(at 156.21 90.17 0)
+			(at 163.83 90.17 0)
 			(effects
 				(font
@@
 		)
 		(property "Description" "Power symbol creates a global label with name \"GND\" , ground"
-			(at 156.21 90.17 0)
+			(at 163.83 90.17 0)
 			(effects
 				(font
@@
 	(symbol
 		(lib_id "Connector_Generic:Conn_01x02")
-		(at 161.29 90.17 0)
+		(at 168.91 90.17 0)
 		(mirror x)
 		(unit 1)
@@
 		(dnp no)
 		(property "Reference" "J9"
-			(at 163.83 90.1701 0)
+			(at 171.45 90.1701 0)
 			(effects
 				(font
@@
 		)
 		(property "Value" "+3.3V"
-			(at 163.83 87.6301 0)
+			(at 171.45 87.6301 0)
 			(effects
 				(font
@@
 		)
 		(property "Footprint" "Connector_JST:JST_XA_B02B-XASK-1_1x02_P2.50mm_Vertical"
-			(at 161.29 90.17 0)
+			(at 168.91 90.17 0)
 			(effects
 				(font
@@
 		)
 		(property "Datasheet" "~"
-			(at 161.29 90.17 0)
+			(at 168.91 90.17 0)
 			(effects
 				(font
@@
 		)
 		(property "Description" "Generic connector, single row, 01x02, script generated (kicad-library-utils/schlib/autogen/connector/)"
-			(at 161.29 90.17 0)
-			(effects
-				(font
+			(at 168.91 90.17 0)
+			(effects
+				(font

Commit message: update pcb sch
Parts:
- J10, J8: value +7.4V -> +6V
Connections:
- net 7.4V renamed +6V
Other:
- moved on the sheet: J10
Changed lines of the file:
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@@
 	(generator_version "8.0")
 	(paper "A4")
-	(label "7.4V"
-		(at 134.62 109.22 180)
+	(symbol
+		(lib_id "power:+6V")
+		(at 163.83 109.22 90)
+		(unit 1)
+		(exclude_from_sim no)
+		(in_bom yes)
+		(on_board yes)
+		(dnp no)
 		(fields_autoplaced yes)
-		(effects
-			(font
-				(size 1.27 1.27)
-			)
-			(justify right bottom)
-		)
-	)
-	(label "7.4V"
-		(at 156.21 109.22 180)
-		(fields_autoplaced yes)
-		(effects
-			(font
-				(size 1.27 1.27)
-			)
-			(justify right bottom)
+		(property "Reference" "#PWR065"
+			(at 167.64 109.22 0)
+			(effects
+				(font
+					(size 1.27 1.27)
+				)
+				(hide yes)
+			)
+		)
+		(property "Value" "+6V"
+			(at 160.02 109.2199 90)
+			(effects
+				(font
+					(size 1.27 1.27)
+				)
+				(justify left)
+			)
+		)
+		(property "Footprint" ""
+			(at 163.83 109.22 0)
+			(effects
+				(font
+					(size 1.27 1.27)
+				)
+				(hide yes)
+			)
+		)
+		(property "Datasheet" ""
+			(at 163.83 109.22 0)
+			(effects
+				(font
+					(size 1.27 1.27)
+				)
+				(hide yes)
+			)
+		)
+		(property "Description" "Power symbol creates a global label with name \"+6V\""
+			(at 163.83 109.22 0)
+			(effects
+				(font
+					(size 1.27 1.27)
+				)
+				(hide yes)
+			)
+		)
+		(pin "1"
+		)
+		(instances
+			(project "Avio-BMS"
+				(path "/14e0994b-afc2-4c10-b50d-3efcc006980d/b371f4c8-5a59-4bdf-859b-16f2afd474be"
+					(reference "#PWR065")
+					(unit 1)
+				)
+			)
 		)
 	)
@@
 	)
 	(symbol
+		(lib_id "power:+6V")
+		(at 134.62 109.22 90)
+		(unit 1)
+		(exclude_from_sim no)
+		(in_bom yes)
+		(on_board yes)
+		(dnp no)
+		(fields_autoplaced yes)
+		(property "Reference" "#PWR064"
+			(at 138.43 109.22 0)
+			(effects
+				(font
+					(size 1.27 1.27)
+				)
+				(hide yes)
+			)
+		)
+		(property "Value" "+6V"
+			(at 130.81 109.2199 90)
+			(effects
+				(font
+					(size 1.27 1.27)
+				)
+				(justify left)
+			)
+		)
+		(property "Footprint" ""
+			(at 134.62 109.22 0)
+			(effects
+				(font
+					(size 1.27 1.27)
+				)
+				(hide yes)
+			)
+		)
+		(property "Datasheet" ""
+			(at 134.62 109.22 0)
+			(effects
+				(font
+					(size 1.27 1.27)
+				)
+				(hide yes)
+			)
+		)
+		(property "Description" "Power symbol creates a global label with name \"+6V\""
+			(at 134.62 109.22 0)
+			(effects
+				(font
+					(size 1.27 1.27)
+				)
+				(hide yes)
+			)
+		)
+		(pin "1"
+		)
+		(instances
+			(project "Avio-BMS"
+				(path "/14e0994b-afc2-4c10-b50d-3efcc006980d/b371f4c8-5a59-4bdf-859b-16f2afd474be"
+					(reference "#PWR064")
+					(unit 1)
+				)
+			)
+		)
+	)
+	(symbol
 		(lib_id "power:GND")
 		(at 134.62 111.76 270)
@@
 	(symbol
 		(lib_id "power:GND")
-		(at 156.21 111.76 270)
+		(at 163.83 111.76 270)
 		(unit 1)
 		(exclude_from_sim no)
@@
 		(fields_autoplaced yes)
 		(property "Reference" "#PWR058"
-			(at 149.86 111.76 0)
+			(at 157.48 111.76 0)
 			(effects
 				(font
@@
 		)
 		(property "Value" "GND"
-			(at 152.4 111.7599 90)
+			(at 160.02 111.7599 90)
 			(effects
 				(font
@@
 		)
 		(property "Footprint" ""
-			(at 156.21 111.76 0)
+			(at 163.83 111.76 0)
 			(effects
 				(font
@@
 		)
 		(property "Datasheet" ""
-			(at 156.21 111.76 0)
+			(at 163.83 111.76 0)
 			(effects
 				(font
@@
 		)
 		(property "Description" "Power symbol creates a global label with name \"GND\" , ground"
-			(at 156.21 111.76 0)
+			(at 163.83 111.76 0)
 			(effects
 				(font
@@
 			)
 		)
-		(property "Value" "+7.4V"
+		(property "Value" "+6V"
 			(at 142.24 109.2201 0)
 			(effects
@@
 	(symbol
 		(lib_id "Connector_Generic:Conn_01x02")
-		(at 161.29 111.76 0)
+		(at 168.91 111.76 0)
 		(mirror x)
 		(unit 1)
@@
 		(dnp no)
 		(property "Reference" "J10"
-			(at 163.83 111.7601 0)
-			(effects
-				(font
-					(size 1.27 1.27)
-				)
-				(justify left)
-			)
-		)
-		(property "Value" "+7.4V"
-			(at 163.83 109.2201 0)
+			(at 171.45 111.7601 0)
+			(effects
+				(font
+					(size 1.27 1.27)
+				)
+				(justify left)
+			)
+		)
+		(property "Value" "+6V"
+			(at 171.45 109.2201 0)
 			(effects
 				(font
@@
 		)
 		(property "Footprint" "Connector_JST:JST_XA_B02B-XASK-1_1x02_P2.50mm_Vertical"
-			(at 161.29 111.76 0)
+			(at 168.91 111.76 0)
 			(effects
 				(font
@@
 		)
 		(property "Datasheet" "~"
-			(at 161.29 111.76 0)
+			(at 168.91 111.76 0)
 			(effects
 				(font
@@
 		)
 		(property "Description" "Generic connector, single row, 01x02, script generated (kicad-library-utils/schlib/autogen/connector/)"
-			(at 161.29 111.76 0)
-			(effects
-				(font
+			(at 168.91 111.76 0)
+			(effects
+				(font

Commit message: ad datasheet
Parts:
- renumbered J7 to J6, J8 to J7, J9 to J8, J10 to J9
Changed lines of the file:
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@@
 		(dnp no)
 		(fields_autoplaced yes)
-		(property "Reference" "#PWR065"
+		(property "Reference" "#PWR064"
 			(at 167.64 109.22 0)
 			(effects
@@
 			(project "Avio-BMS"
 				(path "/14e0994b-afc2-4c10-b50d-3efcc006980d/b371f4c8-5a59-4bdf-859b-16f2afd474be"
-					(reference "#PWR065")
+					(reference "#PWR064")
 					(unit 1)
 				)
@@
 		(dnp no)
 		(fields_autoplaced yes)
-		(property "Reference" "#PWR055"
+		(property "Reference" "#PWR059"
 			(at 128.27 90.17 0)
 			(effects
@@
 			(project "Avio-BMS"
 				(path "/14e0994b-afc2-4c10-b50d-3efcc006980d/b371f4c8-5a59-4bdf-859b-16f2afd474be"
-					(reference "#PWR055")
+					(reference "#PWR059")
 					(unit 1)
 				)
@@
 		(dnp no)
 		(fields_autoplaced yes)
-		(property "Reference" "#PWR064"
+		(property "Reference" "#PWR060"
 			(at 138.43 109.22 0)
 			(effects
@@
 			(project "Avio-BMS"
 				(path "/14e0994b-afc2-4c10-b50d-3efcc006980d/b371f4c8-5a59-4bdf-859b-16f2afd474be"
-					(reference "#PWR064")
+					(reference "#PWR060")
 					(unit 1)
 				)
@@
 		(dnp no)
 		(fields_autoplaced yes)
-		(property "Reference" "#PWR056"
+		(property "Reference" "#PWR061"
 			(at 128.27 111.76 0)
 			(effects
@@
 			(project "Avio-BMS"
 				(path "/14e0994b-afc2-4c10-b50d-3efcc006980d/b371f4c8-5a59-4bdf-859b-16f2afd474be"
-					(reference "#PWR056")
+					(reference "#PWR061")
 					(unit 1)
 				)
@@
 		(dnp no)
 		(fields_autoplaced yes)
-		(property "Reference" "#PWR061"
+		(property "Reference" "#PWR058"
 			(at 138.43 87.63 0)
 			(effects
@@
 			(project "Avio-BMS"
 				(path "/14e0994b-afc2-4c10-b50d-3efcc006980d/b371f4c8-5a59-4bdf-859b-16f2afd474be"
-					(reference "#PWR061")
+					(reference "#PWR058")
 					(unit 1)
 				)
@@
 		(on_board yes)
 		(dnp no)
-		(property "Reference" "J7"
+		(property "Reference" "J6"
 			(at 142.24 90.1701 0)
 			(effects
@@
 			(project "Avio-BMS"
 				(path "/14e0994b-afc2-4c10-b50d-3efcc006980d/b371f4c8-5a59-4bdf-859b-16f2afd474be"
-					(reference "J7")
+					(reference "J6")
 					(unit 1)
 				)
@@
 		(dnp no)
 		(fields_autoplaced yes)
-		(property "Reference" "#PWR058"
+		(property "Reference" "#PWR065"
 			(at 157.48 111.76 0)
 			(effects
@@
 			(project "Avio-BMS"
 				(path "/14e0994b-afc2-4c10-b50d-3efcc006980d/b371f4c8-5a59-4bdf-859b-16f2afd474be"
-					(reference "#PWR058")
+					(reference "#PWR065")
 					(unit 1)
 				)
@@
 		(on_board yes)
 		(dnp no)
-		(property "Reference" "J8"
+		(property "Reference" "J7"
 			(at 142.24 111.7601 0)
 			(effects
@@
 			(project "Avio-BMS"
 				(path "/14e0994b-afc2-4c10-b50d-3efcc006980d/b371f4c8-5a59-4bdf-859b-16f2afd474be"
-					(reference "J8")
+					(reference "J7")
 					(unit 1)
 				)
@@
 		(dnp no)
 		(fields_autoplaced yes)
-		(property "Reference" "#PWR057"
+		(property "Reference" "#PWR063"
 			(at 157.48 90.17 0)
 			(effects
@@
 			(project "Avio-BMS"
 				(path "/14e0994b-afc2-4c10-b50d-3efcc006980d/b371f4c8-5a59-4bdf-859b-16f2afd474be"
-					(reference "#PWR057")
+					(reference "#PWR063")
 					(unit 1)
 				)
@@
 		(on_board yes)
 		(dnp no)
-		(property "Reference" "J9"
+		(property "Reference" "J8"
 			(at 171.45 90.1701 0)
 			(effects
@@
 			(project "Avio-BMS"
 				(path "/14e0994b-afc2-4c10-b50d-3efcc006980d/b371f4c8-5a59-4bdf-859b-16f2afd474be"
-					(reference "J9")
+					(reference "J8")
 					(unit 1)
 				)
@@
 		(on_board yes)
 		(dnp no)
-		(property "Reference" "J10"
+		(property "Reference" "J9"
 			(at 171.45 111.7601 0)
 			(effects
@@
 			(project "Avio-BMS"
 				(path "/14e0994b-afc2-4c10-b50d-3efcc006980d/b371f4c8-5a59-4bdf-859b-16f2afd474be"
-					(reference "J10")
-					(unit 1)
-				)
+					(reference "J9")
+					(unit 1)
+				)

Commit message: update sch
Other:
- moved on the sheet: J6, J7, J8, J9
