File: LTC4088.kicad_sch (KiCad schematic)
At the start: 24 parts, among them J6 Conn_01x03_Pin, J7 Conn_01x03_Pin, J8 Conn_01x03_Pin, Q1 Si2333DDS-T1-GE3, Q2 Si2333DDS-T1-GE3, U3 LTC4088EDE-TRPBF

Commit message: update pcb
Parts:
- removed TH1: NTC, symbol Device:Thermistor_NTC
- added R27, R28, R29: 0, Resistor_SMD:R_0603_1608Metric_Pad0.98x0.95mm_HandSolder, symbol Device:R_Small
- renumbered C11 to C27, C12 to C28, C13 to C29, C32 to C30, C20 to C31, C33 to C32, C23 to C33, D1 to D5, J6 to J4, J7 to J5, J8 to J6, Q1 to Q5, Q2 to Q6, R9 to R20, R10 to R21, R11 to R22, R12 to R23, R13 to R24, R14 to R25, R15 to R26, TP2 to TP4, U3 to U4
Connections:
- net GND: now also R29.2
- net NTC: now also R27.1, R28.1, R29.1
- net GATE: now reaches Q6.1 (G), U4.8 (GATE)
- new net NTC1: R27.2
- new net NTC2: R28.2
Other:
- note added: "MainBattery-layerにつながる"

Commit message: update pcb ltc4088kitsui
Parts:
- added R12: 0, Resistor_SMD:R_0603_1608Metric_Pad0.98x0.95mm_HandSolder, symbol Device:R_Small
- renumbered C33 to C10, C27 to C4, C28 to C5, C29 to C6, C30 to C7, C31 to C8, C32 to C9, D5 to D3, L3 to L1, Q5 to Q1, Q6 to Q2, R24 to R10, R29 to R11, R25 to R13, R26 to R14, R20 to R4, R21 to R5, R22 to R6, R23 to R7, R27 to R8, R28 to R9, U4 to U1
Connections:
- net GATE: now also R12.1; no longer Q2.1 (G)
- net V_{OUT}1: no longer C7.2, C9.2, Q2.3 (D), TP4.1, U1.9 (BAT)
- new net: Q2.1 (G), R12.2
- new net Main-Bat: C7.2, C9.2, Q2.3 (D), TP4.1, U1.9 (BAT)
Other:
- moved on the sheet: C10, C7, C8, C9, Q2, R14, TP4

Commit message: update pcb
Other:
- moved on the sheet: C6, J4, J5, J6

Commit message: update pcb sch
Parts:
- removed J4: Conn_01x03_Pin, Connector_PinHeader_2.54mm:PinHeader_1x03_P2.54mm_Vertical, symbol Connector:Conn_01x03_Pin
- added C3: 100u, Capacitor_SMD:C_1206_3216Metric_Pad1.33x1.80mm_HandSolder, symbol Device:C_Small
- C6: value 10u -> 100u; footprint Capacitor_SMD:C_0805_2012Metric_Pad1.18x1.45mm_HandSolder -> Capacitor_SMD:C_1206_3216Metric_Pad1.33x1.80mm_HandSolder
Connections:
- net D0 is gone; now on net GND: U1.13 (D0)
- net D1: now also J6.2 (Pin_2)
- net D2: no longer J6.2 (Pin_2)
- net GND: now also C3.2
- net V_{IN}: now also C3.1

Commit message: ad datasheet
Parts:
- renumbered C4 to C3, C6 to C4, C3 to C6, J5 to J4, J6 to J5, R9 to R10, R10 to R11, R11 to R12, R12 to R13, R13 to R14, R14 to R15, R4 to R5, R5 to R6, R6 to R7, R7 to R8, R8 to R9

Commit message: update
Connections:
- net D1: no longer J5.2 (Pin_2)
- net D2: now also J5.2 (Pin_2)
Changed lines of the file:
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@@
 		)
 	)
-	(label "D1"
+	(label "D2"
 		(at 149.86 149.86 180)
 		(fields_autoplaced yes)

Commit message: update sch
Connections:
- net V_{OUT}1 renamed VOUTS
Changed lines of the file:
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@@
 	(wire
 		(pts
+			(xy 133.35 73.66) (xy 135.89 73.66)
+		)
+		(stroke
+			(width 0)
+			(type default)
+		)
+	)
+	(wire
+		(pts
 			(xy 177.8 78.74) (xy 180.34 78.74)
 		)
@@
 		)
 	)
+	(label "NTC"
+		(at 133.35 73.66 180)
+		(fields_autoplaced yes)
+		(effects
+			(font
+				(size 1.27 1.27)
+			)
+			(justify right bottom)
+		)
+	)
 	(label "GATE"
 		(at 170.18 86.36 0)
@@
 		)
 	)
-	(global_label "Main-Bat"
-		(shape input)
-		(at 251.46 111.76 0)
+	(label "NTC"
+		(at 129.54 101.6 0)
 		(fields_autoplaced yes)
 		(effects
@@
 				(size 1.27 1.27)
 			)
-			(justify left)
-		)
-		(property "Intersheetrefs" "${INTERSHEET_REFS}"
-			(at 263.5165 111.76 0)
-			(effects
-				(font
-					(size 1.27 1.27)
-				)
-				(justify left)
-				(hide yes)
-			)
+			(justify left bottom)
 		)
 	)
-	(global_label "NTC1"
-		(shape output)
-		(at 125.73 114.3 270)
+	(hierarchical_label "VBUS"
+		(shape input)
+		(at 48.26 86.36 180)
 		(fields_autoplaced yes)
 		(effects
@@
 			(justify right)
 		)
-		(property "Intersheetrefs" "${INTERSHEET_REFS}"
-			(at 125.73 122.0628 90)
-			(effects
-				(font
-					(size 1.27 1.27)
-				)
-				(justify right)
-				(hide yes)
+	)
+	(hierarchical_label "VOUTS"
+		(shape output)
+		(at 267.97 81.28 0)
+		(fields_autoplaced yes)
+		(effects
+			(font
+				(size 1.27 1.27)
 			)
+			(justify left)
 		)
 	)
-	(global_label "NTC"
+	(hierarchical_label "NTC1"
 		(shape input)
-		(at 135.89 73.66 180)
+		(at 125.73 114.3 270)
 		(fields_autoplaced yes)
 		(effects
@@
 			(justify right)
 		)
-		(property "Intersheetrefs" "${INTERSHEET_REFS}"
-			(at 129.3367 73.66 0)
-			(effects
-				(font
-					(size 1.27 1.27)
-				)
-				(justify right)
-				(hide yes)
-			)
-		)
 	)
-	(global_label "NTC"
-		(shape input)
-		(at 129.54 101.6 0)
+	(hierarchical_label "Main-Bat"
+		(shape bidirectional)
+		(at 251.46 111.76 0)
 		(fields_autoplaced yes)
 		(effects
@@
 			(justify left)
 		)
-		(property "Intersheetrefs" "${INTERSHEET_REFS}"
-			(at 136.0933 101.6 0)
-			(effects
-				(font
-					(size 1.27 1.27)
-				)
-				(justify left)
-				(hide yes)
-			)
-		)
 	)
-	(global_label "NTC2"
-		(shape output)
+	(hierarchical_label "NTC2"
+		(shape input)
 		(at 130.81 114.3 270)
 		(fields_autoplaced yes)
@@
 			(justify right)
 		)
-		(property "Intersheetrefs" "${INTERSHEET_REFS}"
-			(at 130.81 122.0628 90)
-			(effects
-				(font
-					(size 1.27 1.27)
-				)
-				(justify right)
-				(hide yes)
-			)
-		)
 	)
 	(symbol
@@
 	)
 	(symbol
-		(lib_id "power:VBUS")
-		(at 48.26 86.36 90)
-		(unit 1)
-		(exclude_from_sim no)
-		(in_bom yes)
-		(on_board yes)
-		(dnp no)
-		(fields_autoplaced yes)
-		(property "Reference" "#PWR014"
-			(at 52.07 86.36 0)
-			(effects
-				(font
-					(size 1.27 1.27)
-				)
-				(hide yes)
-			)
-		)
-		(property "Value" "VBUS"
-			(at 44.45 86.3599 90)
-			(effects
-				(font
-					(size 1.27 1.27)
-				)
-				(justify left)
-			)
-		)
-		(property "Footprint" ""
-			(at 48.26 86.36 0)
-			(effects
-				(font
-					(size 1.27 1.27)
-				)
-				(hide yes)
-			)
-		)
-		(property "Datasheet" ""
-			(at 48.26 86.36 0)
-			(effects
-				(font
-					(size 1.27 1.27)
-				)
-				(hide yes)
-			)
-		)
-		(property "Description" "Power symbol creates a global label with name \"VBUS\""
-			(at 48.26 86.36 0)
-			(effects
-				(font
-					(size 1.27 1.27)
-				)
-				(hide yes)
-			)
-		)
-		(pin "1"
-		)
-		(instances
-			(project "Avio-BMS"
-				(path "/14e0994b-afc2-4c10-b50d-3efcc006980d/3c93f837-0667-4863-b5ad-97e598ccbf82"
-					(reference "#PWR014")
-					(unit 1)
-				)
-			)
-		)
-	)
-	(symbol
 		(lib_id "Connector:TestPoint")
 		(at 231.14 104.14 270)
@@
 					(unit 1)
 				)
-			)
-		)
-	)
-	(symbol
-		(lib_id "power:VCC")
-		(at 267.97 81.28 270)
-		(unit 1)
-		(exclude_from_sim no)
-		(in_bom yes)
-		(on_board yes)
-		(dnp no)
-		(property "Reference" "#PWR030"
-			(at 264.16 81.28 0)
-			(effects
-				(font
-					(size 1.27 1.27)
-				)
-				(hide yes)
-			)
-		)
-		(property "Value" "V_{OUT}1"
-			(at 265.43 78.994 90)
-			(effects
-				(font
-					(size 1.27 1.27)
-				)
-				(justify left)
-			)
-		)
-		(property "Footprint" ""
-			(at 267.97 81.28 0)
-			(effects
-				(font
-					(size 1.27 1.27)
-				)
-				(hide yes)
-			)
-		)
-		(property "Datasheet" ""
-			(at 267.97 81.28 0)
-			(effects
-				(font
-					(size 1.27 1.27)
-				)
-				(hide yes)
-			)
-		)
-		(property "Description" "Power symbol creates a global label with name \"VCC\""
-			(at 267.97 81.28 0)
-			(effects
-				(font
-					(size 1.27 1.27)
-				)
-				(hide yes)
-			)
-		)
-		(pin "1"
-		)
-		(instances
-			(project "Avio-BMS"
-				(path "/14e0994b-afc2-4c10-b50d-3efcc006980d/3c93f837-0667-4863-b5ad-97e598ccbf82"
-					(reference "#PWR030")
-					(unit 1)
-				)

Commit message: 値の更新とテキストボックスの修正; LTC4088およびLTC4417の新しいテキスト追加
Parts:
- R14: value R -> 1k
Changed lines of the file:
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@@
 			)
 		)
-		(property "Value" "R"
+		(property "Value" "1k"
 			(at 223.52 133.35 90)
 			(effects
